File: KiCAD-project-files/slidrr-cy8c.kicad_sch (KiCad schematic)
At the start: 118 parts, among them J1 ISSP U1, J2 ISSP U2, J3 Conn_01x32_Socket, J4 JST-XH Series, J5 JST-XH Series, SW1 SW_DIP_x04, SW2 SW_Push, SW3 SW_Push, U5 SN74LV1T34DBVR

Commit message: Edited PCB to fix floating UART issue. Added crappy WebUI for diagnosis
Connections:
- net at U2.1 (P0[7]): no longer C3.2
Other:
- note added: "SSOP-28 Footprint"
- moved on the sheet: C1, C2, C3, C4, C5, C6, J4, J5, R1, R2, SW1, SW2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
